File: PCB/Modular-Control-Module/Modular-Control-Module.kicad_sch (KiCad schematic)
At the start: 40 parts, among them J1 Conn_ARM_SWD_TagConnect_TC203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, J2 DX07S016JA1R1500, SW1 B3U-1000P, SW2 B3U-1000P, T1 5051101092, U1 TEMPLATE, U2 RP2040, X1 ABM8G-12.000MHZ-18-D2Y-T

Commit message: Schematic Tweak and Board Route
Schaemtic and design tweaked to be SPI only. added more power pins for more current. Finished PCB route only needs to be put through DRC.
Connections:
- net +3.3V: now also T1.2
- net SLAVE_IRQ: now also T1.7; no longer T1.4
- net SPI_CS: now also T1.5; no longer T1.6
- net SPI_MISO: now also T1.4; no longer T1.7
- net SPI_SCK: now also T1.6; no longer T1.5
- net I2C_SCL: no longer names the net of T1.3
- net I2C_SCL: no longer U2.13 (GPIO10)
- net I2C_SDA: no longer names the net of U2.12 (GPIO9)
- net I2C_SDA: no longer T1.2
